File: loggerhw_v5.0.sch (KiCad schematic (older format))
At the start: 64 parts, among them J1 PinHeader_2x08_P1.27mm_Vertic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, J10 PROBE, J11 Conn_01x01_Female, J12 Conn_01x10_Male, J2 Conn_01x06, J20 U.FL-R-SMT-1, J3 Conn_01x06, J4 PinHeader_2x08_P1.27mm_Vertic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, J5 Conn_01x01_Female, J6 Conn_01x01_Female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

Commit message: Version 5.0 added LoRa base station provisions: SD card slot with load switch, expansion header, SMA connector and general improvements
Parts:
- removed C16: DNP - 12pF, Capacitor_SMD:C_0402_1005Metric, symbol Device:C_Small
- removed J1, J4: PinHeader_2x08_P1.27mm_Vertical_SMD, Connector_PinHeader_1.27mm:PinHeader_2x08_P1.27mm_Vertical_SMD, symbol Connector_Generic:Conn_02x08_Odd_Even
- removed R2, R3: DNP, Resistor_SMD:R_0402_1005Metric, symbol Device:R_Small
- removed R4: 0, Resistor_SMD:R_0402_1005Metric, symbol Device:R_Small
- removed Y2: DNP - 32.768Khz, Crystal:Crystal_SMD_3215-2Pin_3.2x1.5mm, symbol Device:Crystal_Small
- added J1: Micro_SD_Card_TF-01, loggerhw_v5:TF-01A, symbol Connector:Micro_SD_Card_TF-01
- added J4: DNP, Connector_PinHeader_2.54mm:PinHeader_1x18_P2.54mm_Vertical, symbol Connector:Conn_01x18_Male
- added J9: DNP, Connector_Coaxial:SMA_Samtec_SMA-J-P-X-ST-EM1_EdgeMount, symbol Connector:Conn_Coaxial
- added U9: TPS22919, Package_TO_SOT_SMD:Texas_R-PDSO-G6, symbol parts:TPS22919
- C1: value DNP - 12pF -> 0.1uF
- R1: value 0 -> DNP
Connections:
- net labels removed: VCC_EXTERNAL, VCC_EXTERNAL2
- wire segments 329 -> 311
- no-connect marks 14 -> 16
Other:
- moved on the sheet: J2, J3
