File: loggerhw_v5.0.kicad_pcb (KiCad board)
At the start: 4 copper layers, 46.5 x 67.8 mm, 62 parts, among them J1 Micro_SD_Card_TF-01, J10 PROBE, J11 Conn_01x01_Female, J12 Conn_01x10_Male, J2 Conn_01x06, J20 U.FL-R-SMT-1, J3 Conn_01x06, J4 DNP, J5 Conn_01x01_Female, J6 Conn_01x01_Female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

Commit message: silk screen tweak
Other:
- net class 50ohm removed
- net class Default removed
- net class Power removed
- board text added: "Licensed under CC BY-NC 4.0 License"
